File: Eagle files/LogicLab1G.brd (EAGLE design)
At the start: 139.7 x 91.4 mm, 153 parts, among them IC1 74AHC1G00DBV, IC10 74AHC1G00DBV, IC11 74AHC1G00DBV, IC12 74AHC1G00DBV, IC13 74AHC1G00DBV, IC14 74AHC1G00DBV, IC15 74AHC1G00DBV, IC16 74AHC1G00DBV, IC17 74AHC1G00DBV, IC2 74AHC1G00DBV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

Commit message: Version 1a - 17th June 2024
Corrected the part numbers of the logic gates.
Parts:
- IC1, IC2: value 74AHC1G00DBV -> 74AHC1G08DBV
- IC10, IC9: value 74AHC1G00DBV -> 74AHC1G86DBV
- IC5, IC6: value 74AHC1G00DBV -> 74AHC1G32DBV
- IC7, IC8: value 74AHC1G00DBV -> 74AHC1G02DBV
Changed lines of the file:
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@@
 <attribute name="PROD_ID" value="DIO-09886" x="11.1125" y="81.28" size="1.778" layer="28" rot="MR270" display="off"/>
 </element>
-<element name="IC1" library="74xx-little-de" package="SOT23-5" value="74AHC1G00DBV" x="35.56" y="71.12" smashed="yes" rot="MR90">
+<element name="IC1" library="74xx-little-de" package="SOT23-5" value="74AHC1G08DBV" x="35.56" y="71.12" smashed="yes" rot="MR90">
 <attribute name="NAME" x="36.83" y="73.66" size="1.27" layer="26" rot="MR0"/>
 </element>
-<element name="IC2" library="74xx-little-de" package="SOT23-5" value="74AHC1G00DBV" x="35.56" y="53.34" smashed="yes" rot="MR90">
+<element name="IC2" library="74xx-little-de" package="SOT23-5" value="74AHC1G08DBV" x="35.56" y="53.34" smashed="yes" rot="MR90">
 <attribute name="NAME" x="36.83" y="55.88" size="1.27" layer="26" rot="MR0"/>
 </element>
@@
 <attribute name="NAME" x="36.83" y="20.32" size="1.27" layer="26" rot="MR0"/>
 </element>
-<element name="IC5" library="74xx-little-de" package="SOT23-5" value="74AHC1G00DBV" x="69.85" y="71.12" smashed="yes" rot="MR90">
+<element name="IC5" library="74xx-little-de" package="SOT23-5" value="74AHC1G32DBV" x="69.85" y="71.12" smashed="yes" rot="MR90">
 <attribute name="NAME" x="71.12" y="73.66" size="1.27" layer="26" rot="MR0"/>
 </element>
-<element name="IC6" library="74xx-little-de" package="SOT23-5" value="74AHC1G00DBV" x="69.85" y="53.34" smashed="yes" rot="MR90">
+<element name="IC6" library="74xx-little-de" package="SOT23-5" value="74AHC1G32DBV" x="69.85" y="53.34" smashed="yes" rot="MR90">
 <attribute name="NAME" x="71.12" y="55.88" size="1.27" layer="26" rot="MR0"/>
 </element>
-<element name="IC7" library="74xx-little-de" package="SOT23-5" value="74AHC1G00DBV" x="69.85" y="35.56" smashed="yes" rot="MR90">
+<element name="IC7" library="74xx-little-de" package="SOT23-5" value="74AHC1G02DBV" x="69.85" y="35.56" smashed="yes" rot="MR90">
 <attribute name="NAME" x="71.12" y="38.1" size="1.27" layer="26" rot="MR0"/>
 </element>
-<element name="IC8" library="74xx-little-de" package="SOT23-5" value="74AHC1G00DBV" x="69.85" y="17.78" smashed="yes" rot="MR90">
+<element name="IC8" library="74xx-little-de" package="SOT23-5" value="74AHC1G02DBV" x="69.85" y="17.78" smashed="yes" rot="MR90">
 <attribute name="NAME" x="71.12" y="20.32" size="1.27" layer="26" rot="MR0"/>
 </element>
-<element name="IC9" library="74xx-little-de" package="SOT23-5" value="74AHC1G00DBV" x="104.14" y="71.12" smashed="yes" rot="MR90">
+<element name="IC9" library="74xx-little-de" package="SOT23-5" value="74AHC1G86DBV" x="104.14" y="71.12" smashed="yes" rot="MR90">
 <attribute name="NAME" x="105.41" y="73.66" size="1.27" layer="26" rot="MR0"/>
 </element>
-<element name="IC10" library="74xx-little-de" package="SOT23-5" value="74AHC1G00DBV" x="104.14" y="53.34" smashed="yes" rot="MR90">
+<element name="IC10" library="74xx-little-de" package="SOT23-5" value="74AHC1G86DBV" x="104.14" y="53.34" smashed="yes" rot="MR90">
 <attribute name="NAME" x="106.68" y="55.88" size="1.27" layer="26" rot="MR0"/>
 </element>
